File: boards/TV-B-Gone-kit-master/pcb_andy/tvbgone3.brd (EAGLE design)
At the start: 22 parts, among them Q5 MPS2907A, U2 ATTINY85V-10SU, Y1 8MHZ

Commit message: board ready for printing
Parts:
- removed +, -: (no value), ybox2:1X01
- removed D1, D2, D3, D4: (no value), SparkFun-LED:LTE-302
- removed ISP1: AVRISP-6, adafruit-edited:AVRISP
- removed LED6: (no value), homemade-hardware:LED-0603
- removed Q5: MPS2907A, transistor-pnp:TO92-CBE
- removed Q6, Q7: (no value), Tomorrow_Lab_LLC:SOT-23-R
- removed R7: 10k, homemade-hardware:0603-RES
- removed R8: 1k, homemade-hardware:0603-RES
- removed U$1: EVP-AVAA1A, Tomorrow_Lab_LLC:EVP-AVAA1A
- added C3, C4, C5, C6: (no value), homemade-hardware:0603-CAP
- added LED1, LED2, LED3: LED, tvbgone:5MM-SIDE
- added LED4: (no value), homemade-hardware:LED-0603
- added Q1: PMBT3906, SparkFun-DiscreteSemi:SOT23-3
- added Q2: (no value), Tomorrow_Lab_LLC:SOT-23-R
- added R1: 10k, homemade-hardware:0603-RES
- added S1: (no value), SparkFun-Electromechanical:TACTILE-SWITCH-SMD
- added TP3, TP4, TP5, TP6: TEST-POINT3X5, SparkFun-Passives:PAD.03X.05
- added TP7, TP8: (no value), microbuilder:TESTPOINT_PAD_2MM
- C1: value 0.1uF -> (none); device rcl-ez:C025-025X050 -> homemade-hardware:0603-CAP
- C2: value 100uF -> (none); device rcl-ez:E2,5-5 -> homemade-hardware:0603-CAP
- moved R6 78.1 mm to (17.6, 17.0), turned to 270 degrees
- moved Q9 72.8 mm to (11.2, 18.4)
- moved R4 69.4 mm to (2.95, 12.9), turned to 90 degrees
- moved Q8 69.3 mm to (7.78, 18.4)
- moved Y1 43.6 mm to (17.5, 11.6), turned to 270 degrees
- moved U2 33.6 mm to (11.3, 11.6), turned to 180 degrees
- moved C2 22.2 mm to (2.37, 7.90), turned to 0 degrees
- moved C1 21.3 mm to (2.37, 6.38), turned to 0 degrees
Connections:
- removed net N$8: D2.C, Q7.2-COLLECTOR
- net GND: now also C2.2, C3.2, C4.2, C5.2, C6.2, Q2.3-EMITTER, S1.1, S1.2, TP7.P$1; no longer -.1, C2.-, ISP1.6, Q6.3-EMITTER, Q7.3-EMITTER, R7.1, U$1.P$1, U$1.P$2
- net MISO: now also TP4.P$1; no longer ISP1.1, R7.2
- net MOSI: now also TP5.P$1; no longer ISP1.4
- net N$10: now also Q1.3, Q2.1-BASE; no longer Q5.C, Q6.1-BASE, Q7.1-BASE
- net N$3: now also LED4.C, R1.2; no longer LED6.C, R8.1
- net N$4: now also LED1.K, LED1.K2, Q2.2-COLLECTOR; no longer D1.C, Q6.2-COLLECTOR
- net N$5: now also LED2.K, LED2.K2, Q8.2-COLLECTOR; no longer D4.C, Q9.2-COLLECTOR
- net N$6: now also Q1.1; no longer Q5.B
- net N$7: now also LED3.K, LED3.K2, Q9.2-COLLECTOR; no longer D3.C, Q8.2-COLLECTOR
- net RST: now also S1.3, S1.4, TP3.P$1; no longer ISP1.5, U$1.P$3, U$1.P$4
- net SCK: now also R1.1, TP6.P$1; no longer ISP1.3, R8.2
- net VCC: now also C2.1, C3.1, C4.1, C5.1, C6.1, LED1.A, LED1.A2, LED2.A, LED2.A2, LED3.A, LED3.A2, LED4.A, Q1.2, TP8.P$1; no longer +.1, C2.+, D1.A, D2.A, D3.A, D4.A, ISP1.2, LED6.A, Q5.E
Routing:
- net VCC: track 0.00 -> 96.7 mm
- net N$10: track 0.00 -> 17.7 mm
- net RST: track 0.00 -> 9.97 mm
- net SCK: track 0.00 -> 9.28 mm
- net N$5: track 0.00 -> 7.49 mm
- net N$6: track 0.00 -> 6.38 mm
- net MOSI: track 0.00 -> 5.25 mm
- net N$7: track 0.00 -> 4.68 mm
- net N$4: track 0.00 -> 4.60 mm
- net MISO: track 0.00 -> 3.71 mm
- net N$1: track 0.00 -> 2.61 mm
- net N$2: track 0.00 -> 2.61 mm
- net N$3: track 0.00 -> 1.78 mm
- added copper zone on layer 1, net GND
Other:
- board outline added: 22.1 x 28.3 mm
