File: boards/TV-B-Gone-kit-master/pcb_andy/tvbgone3.sch (EAGLE design)
At the start: 22 parts, among them Q5 MPS2907A, U2 ATTINY85V-10SU, Y1 8MHZ

Commit message: board ready for printing
Parts:
- removed +, -: (no value), ybox2:PINHD-1X1
- removed D1, D2, D3, D4: (no value), SparkFun-LED:LTE-302
- removed ISP1: AVRISP-6, adafruit-edited:AVRISP-6
- removed LED6: (no value), homemade-hardware:LED0603
- removed Q5: MPS2907A, transistor-pnp:MPS2907A
- removed Q6, Q7: (no value), Tomorrow_Lab_LLC:TRANSISTOR_NPN
- removed R7: 10k, homemade-hardware:RESISTOR0603
- removed R8: 1k, homemade-hardware:RESISTOR0603
- removed U$1: EVP-AVAA1A, Tomorrow_Lab_LLC:EVP-AVAA1A
- added C3, C4, C5, C6: (no value), homemade-hardware:CAP0603-CAP
- added LED1, LED2, LED3: LED, tvbgone:LED
- added LED4: (no value), homemade-hardware:LED0603
- added Q1: PMBT3906, SparkFun-DiscreteSemi:TRANSISTOR_PNPPMBT3906
- added Q2: (no value), Tomorrow_Lab_LLC:TRANSISTOR_NPN
- added R1: 10k, homemade-hardware:RESISTOR0603
- added S1: (no value), SparkFun-Electromechanical:TAC_SWITCHSMD
- added TP3, TP4, TP5, TP6: TEST-POINT3X5, SparkFun-Passives:TEST-POINT3X5
- added TP7, TP8: (no value), microbuilder:TESTPOINTPAD
- C1: value 0.1uF -> (none); device rcl-ez:C-US025-025X050 -> homemade-hardware:CAP0603-CAP
- C2: value 100uF -> (none); device rcl-ez:CPOL-USE2.5-5 -> homemade-hardware:CAP0603-CAP
Connections:
- removed net N$8: D2.C, Q7.C
- net GND: now also C2.2, C3.2, C4.2, C5.2, C6.2, Q2.E, S1.1, S1.2, TP7.P$1; no longer -.1, C2.-, ISP1.GND, Q6.E, Q7.E, R7.1, U$1.1
- net MISO: now also TP4.1; no longer ISP1.MISO, R7.2
- net MOSI: now also TP5.1; no longer ISP1.MOSI
- net N$10: now also Q1.C, Q2.B; no longer Q5.C, Q6.B, Q7.B
- net N$3: now also LED4.C, R1.2; no longer LED6.C, R8.1
- net N$4: now also LED1.C, LED1.C1, Q2.C; no longer D1.C, Q6.C
- net N$5: now also LED2.C, LED2.C1, Q8.C; no longer D4.C, Q9.C
- net N$6: now also Q1.B; no longer Q5.B
- net N$7: now also LED3.C, LED3.C1, Q9.C; no longer D3.C, Q8.C
- net RST: now also S1.3, S1.4, TP3.1; no longer ISP1.RST, U$1.2
- net SCK: now also R1.1, TP6.1; no longer ISP1.SCK, R8.2
- net VCC: now also C2.1, C3.1, C4.1, C5.1, C6.1, LED1.A, LED1.A1, LED2.A, LED2.A1, LED3.A, LED3.A1, LED4.A, Q1.E, TP8.P$1; no longer +.1, C2.+, D1.A, D2.A, D3.A, D4.A, ISP1.VCC, LED6.A, Q5.E
Other:
- note added: "avrdude -c avrisp2 -p attiny85 -D -U lfuse:w:0xfe avrdude -c avrisp2 -p attiny85 -D -U hfuse:w:0xdf avrdude -c avrisp2 -p attiny85 -D -U efuse:w:0xff avrdude -c avrisp2 -p attiny85 -D -U flash:w:path/to/image.hex"
- note removed: "Battery"
- moved on the sheet: C1
