File: boards/TV-B-Gone-kit-master/pcb_andy_4/tvbgone.brd (EAGLE design)
At the start: 25.5 x 39.5 mm, 34 parts, among them U1 ATMEGA328P, Y1 18MHZ

Commit message: about to populate panels at ITP
Parts:
- added C10, C11, C8, C9: 4.7uF, homemade-hardware:0603-CAP
- moved R1 3.01 mm to (20.5, 23.9), turned to 270 degrees
- moved R6 1.41 mm to (15.9, 23.9)
- moved LED4 0.92 mm to (18.2, 23.9)
- moved C1 0.90 mm to (23.6, 23.6)
- moved C4 0.90 mm to (23.6, 25.1)
- moved C6 0.90 mm to (23.6, 22.1)
- moved C3 0.80 mm to (12.9, 25.0)
- moved C2 0.80 mm to (12.9, 23.6)
- moved C5 0.80 mm to (12.9, 22.1)
- moved Q2 0.50 mm to (16.2, 27.6)
- moved Q9 0.50 mm to (20.2, 27.6)
- moved R10 0.30 mm to (12.7, 30.8)
- moved R8 0.30 mm to (23.8, 30.8)
- moved R7 0.20 mm to (22.6, 30.8)
- moved R12 0.20 mm to (13.9, 30.8)
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Connections:
- net GND: now also C10.2, C11.2, C8.2, C9.2
- net VCC: now also C10.1, C11.1, C8.1, C9.1
Routing:
- net VCC: track 124.0 -> 116.5 mm
- net GND: track 21.3 -> 19.7 mm
- net N$3: track 1.39 -> 2.80 mm
- net N$10: track 12.9 -> 14.0 mm
- net N$11: track 5.80 -> 6.41 mm
- net N$4: track 5.80 -> 6.36 mm
