File: boards/power/lipo_charger/lipo_charger.brd (EAGLE design)
At the start: 11.9 x 31.2 mm, 11 parts, among them IC1 MCP73831/OT

Commit message: prep lipo board for class 6
Parts:
- R1, R2: value 1k -> 470
