File: boards/power/lipo_charger/lipo_charger.sch (EAGLE design)
At the start: 11 parts, among them IC1 MCP73831/OT

Commit message: prep lipo board for class 6
Parts:
- R1, R2: value 1k -> 470
Other:
- note removed: "LiPo Charger IC - digikey # MCP73831T-2ACI/OTCT-ND"
- moved on the sheet: BATTERY, C1, C2, CHARGING, DONE, R1, R2
