File: projects/eagle-board-design/1_attiny85_jig/attiny85_jig.sch (EAGLE design)
At the start: 6 parts

Commit message: gives names to connections in jig pcb
Connections:
- net N$1 renamed MOSI
- net N$2 renamed MISO
- net N$3 renamed SCK
- net N$4 renamed ARDUINO_RESET
- net RESET renamed TINY_RESET
Changed lines of the file:
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@@
 </busses>
 <nets>
-<net name="RESET" class="0">
+<net name="TINY_RESET" class="0">
 <segment>
 <pinref part="U$1" gate="G$1" pin="RESET_(PB5)"/>
@@
 </segment>
 </net>
-<net name="N$1" class="0">
+<net name="MOSI" class="0">
 <segment>
 <pinref part="U$1" gate="G$1" pin="D0_MOSI_(PB0)"/>
@@
 </segment>
 </net>
-<net name="N$2" class="0">
+<net name="MISO" class="0">
 <segment>
 <pinref part="U$1" gate="G$1" pin="D1_MISO_(PB1)"/>
@@
 </segment>
 </net>
-<net name="N$3" class="0">
+<net name="SCK" class="0">
 <segment>
 <pinref part="U$1" gate="G$1" pin="A1/D2_SCK_(PB2)"/>
@@
 </segment>
 </net>
-<net name="N$4" class="0">
+<net name="ARDUINO_RESET" class="0">
 <segment>
 <pinref part="U$2" gate="G$1" pin="6"/>
