File: examples/lipo-charger/lipo-charger.sch (EAGLE design)
At the start: 10 parts, among them IC2 LIPO_CHARGER/OT

Commit message: lipo board uses new parts
Parts:
- removed CN1: (no value), homemade-hardware:JST_2PIN_BATTERY-SMT-HORIZ
- removed IC2: LIPO_CHARGER/OT, homemade-hardware:LIPO_CHARGER/OT
- added IC1: IC_LIPO_CHARGER, homemade-hardware:IC_LIPO_CHARGER
- added U$1: CONN_BATTERY-LIPO-HORIZ, homemade-hardware:CONN_BATTERY-LIPO-HORIZ
- C1, C2: device homemade-hardware:CAP-0805 -> homemade-hardware:COMPONENT_CAP-0805
- LED1: value RED-2V/20mA -> Red
- LED2: value GREEN-2V/20mA -> Blue
- R1: value 10k -> 150; device homemade-hardware:RESISTOR-0805 -> homemade-hardware:COMPONENT_RESISTOR-0805
- R2: device homemade-hardware:RESISTOR-0805 -> homemade-hardware:COMPONENT_RESISTOR-0805
- R3: value 150 -> 10k; device homemade-hardware:RESISTOR-0805 -> homemade-hardware:COMPONENT_RESISTOR-0805
- U$2: value USB-PCB-POWER -> CONN_USB_PCB_POWER; device homemade-hardware:USB-PCB-POWER -> homemade-hardware:CONN_USB_PCB_POWER
Connections:
- net 5V: now also IC1.VDD; no longer IC2.VDD
- net BATTERY: now also IC1.VBAT, U$1.+; no longer CN1.2, IC2.VBAT
- net CURRENT-CONTROL: now also IC1.PROG, R3.2; no longer IC2.PROG, R1.2
- net GND: now also IC1.GND, R3.1, U$1.-; no longer CN1.1, IC2.VSS, R1.1
- net N$2: now also R1.2; no longer R2.2
- net N$3: now also R2.1; no longer R3.1
- net STATUS: now also IC1.STAT, R1.1, R2.2; no longer IC2.STAT, R2.1, R3.2
Other:
- moved on the sheet: R1, R2, R3

Commit message: finishes lipo pcb design
Other:
- moved on the sheet: U$2
Changed lines of the file:
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@@
 <part name="IC1" library="homemade-hardware" deviceset="IC_LIPO_CHARGER" device=""/>
 <part name="U$1" library="homemade-hardware" deviceset="CONN_BATTERY" device="-LIPO-HORIZ"/>
-<part name="GND7" library="homemade-hardware" deviceset="GND" device=""/>
-<part name="GND8" library="homemade-hardware" deviceset="GND" device=""/>
-<part name="GND9" library="homemade-hardware" deviceset="GND" device=""/>
-<part name="GND10" library="homemade-hardware" deviceset="GND" device=""/>
-<part name="GND11" library="homemade-hardware" deviceset="GND" device=""/>
-<part name="GND12" library="homemade-hardware" deviceset="GND" device=""/>
 <part name="U$2" library="homemade-hardware" deviceset="CONN_USB_PCB_POWER" device=""/>
 <part name="LED1" library="homemade-hardware" deviceset="LED" device="-0805" value="Red"/>
@@
 <part name="R1" library="homemade-hardware" deviceset="COMPONENT_RESISTOR" device="-0805" value="150"/>
 <part name="R3" library="homemade-hardware" deviceset="COMPONENT_RESISTOR" device="-0805" value="10k"/>
+<part name="GND1" library="homemade-hardware" deviceset="SYMBOL_GND" device=""/>
+<part name="GND2" library="homemade-hardware" deviceset="SYMBOL_GND" device=""/>
+<part name="GND3" library="homemade-hardware" deviceset="SYMBOL_GND" device=""/>
+<part name="GND4" library="homemade-hardware" deviceset="SYMBOL_GND" device=""/>
+<part name="GND5" library="homemade-hardware" deviceset="SYMBOL_GND" device=""/>
+<part name="GND6" library="homemade-hardware" deviceset="SYMBOL_GND" device=""/>
 </parts>
 <sheets>
 <sheet>
 <plain>
-<text x="154.94" y="25.4" size="1.778" layer="150">10k    =   100mA
+<text x="149.86" y="15.24" size="1.778" layer="150">10k    =   100mA
 4.7k   =   200mA
 2k      =   500mA
@@
 <instance part="U$1" gate="G$1" x="180.34" y="40.64" smashed="yes">
 <attribute name="NAME" x="182.88" y="49.53" size="1.27" layer="95"/>
-<attribute name="VALUE" x="182.88" y="30.48" size="1.27" layer="96"/>
 </instance>
-<instance part="GND7" gate="1" x="71.12" y="17.78" smashed="yes">
-<attribute name="VALUE" x="68.58" y="15.24" size="1.778" layer="96"/>
-</instance>
-<instance part="GND8" gate="1" x="58.42" y="48.26" smashed="yes">
-<attribute name="VALUE" x="55.88" y="45.72" size="1.778" layer="96"/>
-</instance>
-<instance part="GND9" gate="1" x="144.78" y="17.78" smashed="yes">
-<attribute name="VALUE" x="142.24" y="15.24" size="1.778" layer="96"/>
-</instance>
-<instance part="GND10" gate="1" x="180.34" y="17.78" smashed="yes">
-<attribute name="VALUE" x="177.8" y="15.24" size="1.778" layer="96"/>
-</instance>
-<instance part="GND11" gate="1" x="99.06" y="40.64" smashed="yes">
-<attribute name="VALUE" x="96.52" y="38.1" size="1.778" layer="96"/>
-</instance>
-<instance part="GND12" gate="1" x="109.22" y="40.64" smashed="yes">
-<attribute name="VALUE" x="106.68" y="38.1" size="1.778" layer="96"/>
-</instance>
-<instance part="U$2" gate="G$1" x="53.34" y="60.96" smashed="yes" rot="MR0">
-<attribute name="NAME" x="55.88" y="64.77" size="1.27" layer="95" rot="MR0"/>
-<attribute name="VALUE" x="55.88" y="53.34" size="1.27" layer="96" rot="MR0"/>
+<instance part="U$2" gate="G$1" x="71.12" y="60.96" smashed="yes" rot="MR0">
+<attribute name="NAME" x="73.66" y="64.77" size="1.27" layer="95" rot="MR0"/>
 </instance>
 <instance part="LED1" gate="G$1" x="86.36" y="53.34" smashed="yes">
@@
 <attribute name="VALUE" x="155.702" y="29.21" size="1.778" layer="96" rot="R90"/>
 </instance>
+<instance part="GND1" gate="1" x="76.2" y="48.26" smashed="yes"/>
+<instance part="GND2" gate="1" x="71.12" y="17.78" smashed="yes"/>
+<instance part="GND3" gate="1" x="99.06" y="40.64" smashed="yes"/>
+<instance part="GND4" gate="1" x="109.22" y="40.64" smashed="yes"/>
+<instance part="GND5" gate="1" x="144.78" y="17.78" smashed="yes"/>
+<instance part="GND6" gate="1" x="180.34" y="17.78" smashed="yes"/>
 </instances>
 <busses>
@@
 <segment>
 <wire x1="86.36" y1="58.42" x2="86.36" y2="55.88" width="0.1524" layer="91"/>
-<wire x1="58.42" y1="58.42" x2="86.36" y2="58.42" width="0.1524" layer="91"/>
+<wire x1="76.2" y1="58.42" x2="86.36" y2="58.42" width="0.1524" layer="91"/>
 <junction x="86.36" y="58.42"/>
 <wire x1="86.36" y1="58.42" x2="99.06" y2="58.42" width="0.1524" layer="91"/>
@@
 <net name="GND" class="0">
 <segment>
-<wire x1="180.34" y1="27.94" x2="180.34" y2="20.32" width="0.1524" layer="91"/>
-<pinref part="U$1" gate="G$1" pin="-"/>
-<pinref part="GND10" gate="1" pin="GND"/>
+<wire x1="76.2" y1="55.88" x2="76.2" y2="50.8" width="0.1524" layer="91"/>
+<pinref part="U$2" gate="G$1" pin="GND"/>
+<pinref part="GND1" gate="1" pin="GND"/>
+</segment>
+<segment>
+<wire x1="71.12" y1="22.86" x2="71.12" y2="20.32" width="0.1524" layer="91"/>
+<pinref part="LED2" gate="G$1" pin="C"/>
+<pinref part="GND2" gate="1" pin="GND"/>
+</segment>
+<segment>
+<wire x1="99.06" y1="45.72" x2="99.06" y2="43.18" width="0.1524" layer="91"/>
+<pinref part="C1" gate="G$1" pin="2"/>
+<pinref part="GND3" gate="1" pin="GND"/>
+</segment>
+<segment>
+<wire x1="109.22" y1="45.72" x2="109.22" y2="43.18" width="0.1524" layer="91"/>
+<pinref part="C2" gate="G$1" pin="2"/>
+<pinref part="GND4" gate="1" pin="GND"/>
 </segment>
 <segment>
@@
 <junction x="144.78" y="27.94"/>
 <pinref part="IC1" gate="G$1" pin="GND"/>
-<pinref part="GND9" gate="1" pin="GND"/>
 <pinref part="R3" gate="G$1" pin="1"/>
+<pinref part="GND5" gate="1" pin="GND"/>
 </segment>
 <segment>
-<wire x1="71.12" y1="22.86" x2="71.12" y2="20.32" width="0.1524" layer="91"/>
-<pinref part="GND7" gate="1" pin="GND"/>
-<pinref part="LED2" gate="G$1" pin="C"/>
-</segment>
-<segment>
-<wire x1="58.42" y1="55.88" x2="58.42" y2="50.8" width="0.1524" layer="91"/>
-<pinref part="GND8" gate="1" pin="GND"/>
-<pinref part="U$2" gate="G$1" pin="GND"/>
-</segment>
-<segment>
-<wire x1="99.06" y1="45.72" x2="99.06" y2="43.18" width="0.1524" layer="91"/>
-<pinref part="GND11" gate="1" pin="GND"/>
-<pinref part="C1" gate="G$1" pin="2"/>
-</segment>
-<segment>
-<wire x1="109.22" y1="45.72" x2="109.22" y2="43.18" width="0.1524" layer="91"/>
-<pinref part="GND12" gate="1" pin="GND"/>
-<pinref part="C2" gate="G$1" pin="2"/>
+<wire x1="180.34" y1="27.94" x2="180.34" y2="20.32" width="0.1524" layer="91"/>
+<pinref part="U$1" gate="G$1" pin="-"/>
+<pinref part="GND6" gate="1" pin="GND"/>
 </segment>
 </net>
