File: examples/microcontrollers/ATSAMD11C14A/eagle/ATSAMD11C14A.sch (EAGLE design)
At the start: 7 parts, among them U1 MICRO_ATSAMD11C14-

Commit message: marquee template; schematic images
Connections:
- net RESET renamed RESET_SAMD11
Other:
- moved on the sheet: C1
Changed lines of the file:
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@@
 <instance part="GND4" gate="1" x="15.24" y="66.04" smashed="yes"/>
 <instance part="GND5" gate="1" x="60.96" y="63.5" smashed="yes"/>
-<instance part="GND1" gate="1" x="5.08" y="17.78" smashed="yes"/>
+<instance part="GND1" gate="1" x="2.54" y="17.78" smashed="yes"/>
 <instance part="GND6" gate="1" x="86.36" y="17.78" smashed="yes"/>
 <instance part="U$4" gate="G$1" x="7.62" y="76.2" smashed="yes" rot="MR0"/>
 <instance part="P+4" gate="G$1" x="88.9" y="78.74" smashed="yes"/>
-<instance part="P+5" gate="G$1" x="5.08" y="53.34" smashed="yes"/>
+<instance part="P+5" gate="G$1" x="2.54" y="53.34" smashed="yes"/>
 <instance part="P+1" gate="G$1" x="86.36" y="38.1" smashed="yes"/>
 <instance part="U$2" gate="G$1" x="45.72" y="76.2" smashed="yes"/>
@@
 <attribute name="VALUE" x="25.4" y="20.066" size="1.778" layer="96" align="top-left"/>
 </instance>
-<instance part="C1" gate="G$1" x="5.08" y="33.02" smashed="yes">
-<attribute name="NAME" x="6.604" y="35.941" size="1.778" layer="95"/>
-<attribute name="VALUE" x="6.604" y="30.861" size="1.778" layer="96"/>
+<instance part="C1" gate="G$1" x="2.54" y="33.02" smashed="yes">
+<attribute name="NAME" x="4.064" y="35.941" size="1.778" layer="95"/>
+<attribute name="VALUE" x="4.064" y="30.861" size="1.778" layer="96"/>
 </instance>
 <instance part="U$3" gate="G$1" x="93.98" y="33.02" smashed="yes" rot="R180"/>
@@
 </segment>
 <segment>
-<wire x1="22.86" y1="22.86" x2="5.08" y2="22.86" width="0.1524" layer="91"/>
-<wire x1="5.08" y1="22.86" x2="5.08" y2="20.32" width="0.1524" layer="91"/>
-<junction x="5.08" y="22.86"/>
-<wire x1="5.08" y1="22.86" x2="5.08" y2="30.48" width="0.1524" layer="91"/>
+<wire x1="22.86" y1="22.86" x2="2.54" y2="22.86" width="0.1524" layer="91"/>
+<wire x1="2.54" y1="22.86" x2="2.54" y2="20.32" width="0.1524" layer="91"/>
+<junction x="2.54" y="22.86"/>
+<wire x1="2.54" y1="22.86" x2="2.54" y2="30.48" width="0.1524" layer="91"/>
 <pinref part="GND1" gate="1" pin="GND"/>
 <pinref part="U1" gate="G$1" pin="GND"/>
@@
 </segment>
 </net>
-<net name="RESET" class="0">
-<segment>
-<label x="20.32" y="45.72" size="1.27" layer="95" rot="R180" xref="yes"/>
-<wire x1="22.86" y1="45.72" x2="20.32" y2="45.72" width="0.1524" layer="91"/>
-<pinref part="U1" gate="G$1" pin="RESET"/>
-</segment>
-<segment>
-<wire x1="88.9" y1="30.48" x2="86.36" y2="30.48" width="0.1524" layer="91"/>
-<label x="86.36" y="30.48" size="1.27" layer="95" rot="MR0" xref="yes"/>
-<pinref part="U$3" gate="G$1" pin="2"/>
-</segment>
-</net>
 <net name="VDD" class="0">
 <segment>
-<wire x1="5.08" y1="50.8" x2="5.08" y2="48.26" width="0.1524" layer="91"/>
-<wire x1="22.86" y1="48.26" x2="5.08" y2="48.26" width="0.1524" layer="91"/>
-<junction x="5.08" y="48.26"/>
-<wire x1="5.08" y1="38.1" x2="5.08" y2="48.26" width="0.1524" layer="91"/>
+<wire x1="2.54" y1="50.8" x2="2.54" y2="48.26" width="0.1524" layer="91"/>
+<wire x1="22.86" y1="48.26" x2="2.54" y2="48.26" width="0.1524" layer="91"/>
+<junction x="2.54" y="48.26"/>
+<wire x1="2.54" y1="38.1" x2="2.54" y2="48.26" width="0.1524" layer="91"/>
 <pinref part="P+5" gate="G$1" pin="VDD"/>
 <pinref part="U1" gate="G$1" pin="VCC"/>
@@
 </segment>
 </net>
+<net name="RESET_SAMD11" class="0">
+<segment>
+<label x="20.32" y="45.72" size="1.27" layer="95" rot="R180" xref="yes"/>
+<wire x1="22.86" y1="45.72" x2="20.32" y2="45.72" width="0.1524" layer="91"/>
+<pinref part="U1" gate="G$1" pin="RESET"/>
+</segment>
+<segment>
+<wire x1="88.9" y1="30.48" x2="86.36" y2="30.48" width="0.1524" layer="91"/>
+<label x="86.36" y="30.48" size="1.27" layer="95" rot="MR0" xref="yes"/>
+<pinref part="U$3" gate="G$1" pin="2"/>
+</segment>
+</net>
